File: my_first_audio_player.kicad_pcb (KiCad board)
At the start: 2 copper layers, 68.1 x 55.9 mm, 57 parts, among them J1 B2B-PH-SM4-TB(LF)(SN), J2 USB3090-XX-X_REVE, J3 SJ-3523-SMT-TR, J4 Conn_01x05_Male, J5 Conn_01x05_Male, J6 Conn 2_10_L, J7 Conn 2_10_R, Q1 SI2333CDS-T1-GE3, U1 ADP150TUJZ3.3-EPR2, U2 MCP73826_4.1VCHCT_ND, U3 PCM1793ADB, U4 LTC3245HMSEPBF, U5 OPA2134, U6 LTC1983ES6-5TRMPBF

Commit message: [Minor] Still not edit Switch, ESP32I2S, PinsocketNumber (develop)
Parts:
- removed the C7 at (131.1, 111.8)
- removed the U4 at (131.1, 106.7)
- removed the U5 at (147.3, 95.0)
- added C7: 1uF, Capacitor_SMD:C_0805_2012Metric, F.Cu at (201.7, 57.4)
- added C7: 10uF, Capacitor_SMD:C_0805_2012Metric, F.Cu at (96.2, 72.8)
- added U4: ESP32-WROOM-32, ESP32-WROOM-32:MODULE_ESP32-WROOM-32, F.Cu at (177.1, 53.4)
- added U4: LTC3245HMSEPBF, LTC3245HMSE:MSOP-12_MSE, F.Cu at (143.3, 42.9)
- added U5: OPA2134, OPA2134UA:SOIC127P599X175-8N, F.Cu at (209.1, 43.1)
- added U5: OPA2134, OPA2134UA:SOIC127P599X175-8N, F.Cu at (128.4, 55.2)
- added U7: ADP150TUJZ3.3-EPR2, ADP151:Analog_Devices-ADP151TUJZ3.3-EPR2-Level_A, F.Cu at (190.2, 64.3)
- C11, C12, C13, C14, C15, C16, C21, C22, C23, C8, C9, R10, R11, R12, R13, R14, R15, R16, R17, R4, R5, R6, R7, R8, R9, U3: moved to F.Cu
- J6: value Conn 2_10_L -> B6B-ZR(LF)(SN); footprint SAMTEC-HTSW-110-18-X-D:SAMTEC-HTSW-110-18-X-D -> B6B-ZR_LF_SN:JST_B6B-ZR(LF)(SN)
- J7: value Conn 2_10_R -> MEM2067-02-180-00-A_REVB; footprint SAMTEC-HTSW-110-18-X-D:SAMTEC-HTSW-110-18-X-D -> MEM2067-02-180-00-A_REVB:GCT_MEM2067-02-180-00-A_REVB
- moved J6 111.3 mm to (193.4, 59.6), turned to 0 degrees
- moved J7 109.1 mm to (195.9, 47.9), turned to 0 degrees
- moved J4 89.2 mm to (96.3, 54.2)
- moved C18 85.6 mm to (152.2, 45.8)
- moved U3 75.1 mm to (123.1, 46.0)
- moved J5 74.3 mm to (114.9, 42.5)
- moved C20 73.4 mm to (134.5, 44.5)
- moved C19 73.2 mm to (144.9, 54.3), turned to 0 degrees
- moved C10 72.7 mm to (118.1, 59.3)
- moved U6 69.2 mm to (134.8, 55.9)
- moved C8 68.7 mm to (147.7, 47.2), turned to 0 degrees
- moved U1 68.6 mm to (135.4, 51.4)
- moved C17 67.8 mm to (140.4, 57.3), turned to 0 degrees
- moved U2 65.1 mm to (149.7, 42.2)
- moved C9 64.4 mm to (140.4, 54.3), turned to 0 degrees
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Connections:
- net /-5V renamed /-VCC
- C10 pad 1: /+5V -> /+VCC
- C9 pad 1: /+5V -> /+VCC
- J2 pad 6: (no net) -> GND
- J2 pad 7: (no net) -> GND
- J4 pad 5: /+5V -> /+VCC
- J6 pad 1: /R1L_1 -> GND
- J6 pad 2: /C1L_2 -> /+3V3
- J6 pad 3: /R2L_1 -> /TXD0
- J6 pad 4: /C1L_1 -> /RXD0
- J6 pad 5: /C1L_2 -> /CPU_EN
- J6 pad 6: GND -> /BOOT
- J7 pad 1: /R1R_1 -> /SD_CS
- J7 pad 10: /C2R_1 -> Net-(J7-Pad10)
- J7 pad 11: /C1R_1 -> Net-(J7-Pad10)
- J7 pad 12: /C3R_1 -> Net-(J7-Pad10)
- J7 pad 2: /C1R_2 -> /SD_MOSI
- J7 pad 3: /R2R_1 -> GND
- J7 pad 4: /C1R_1 -> /+3V3
- J7 pad 5: /C1R_2 -> /SD_SCK
- J7 pad 7: /C1R_1 -> /SD_MISO
- J7 pad 8: /C3R_2 -> Net-(J7-Pad8)
- J7 pad 9: /C1R_2 -> Net-(J7-Pad10)
- U3 pad 1: /LRLK -> /LRCK
- U3 pad 10: /+5V -> /+VCC
- U3 pad 15: /+5V -> /+VCC
- U3 pad 20: /+5V -> /+VCC
- U3 pad 21: /+5V -> /+VCC
- U3 pad 26: /+5V -> /+VCC
- U3 pad 28: /+5V -> /+VCC
Routing:
- net GND: vias 3 -> 0
- net /R_OUT: vias 1 -> 0
- net /L_OUT: vias 1 -> 0
- net (no net): vias 4 -> 0

Commit message: [Minor] Maybe create ver2 sch (develop)
Parts:
- removed the C7 at (201.7, 57.4)
- removed the C7 at (96.2, 72.8)
- removed the U4 at (177.1, 53.4)
- removed the U4 at (143.3, 42.9)
- removed the U5 at (209.1, 43.1)
- removed the U5 at (128.4, 55.2)
- added C24: 0.1u, Capacitor_SMD:C_0805_2012Metric, F.Cu at (157.3, 40.4)
- added C25: 0.1u, Capacitor_SMD:C_0805_2012Metric, F.Cu at (152.9, 45.3)
- added C7: 1uF, Capacitor_SMD:C_0805_2012Metric, F.Cu at (136.5, 56.8)
- added R18: 10k, Resistor_SMD:R_0805_2012Metric, F.Cu at (157.3, 49.3)
- added R19: 10k, Resistor_SMD:R_0805_2012Metric, F.Cu at (149.8, 57.2)
- added S2: EG6201, EG6201:SW_EG6201, F.Cu at (99.0, 49.3)
- added S3: 2-1437565-8, 2-1437565-8:SW_2-1437565-8, F.Cu at (143.3, 20.8)
- added S4: 2-1437565-8, 2-1437565-8:SW_2-1437565-8, F.Cu at (143.3, 28.4)
- added S5: 2-1437565-8, 2-1437565-8:SW_2-1437565-8, F.Cu at (94.5, 60.8)
- added S6: 2-1437565-8, 2-1437565-8:SW_2-1437565-8, F.Cu at (107.8, 60.8)
- added U4: ESP32-WROOM-32, ESP32-WROOM-32:MODULE_ESP32-WROOM-32, F.Cu at (98.3, 30.6)
- added U5: OPA2134, OPA2134UA:SOIC127P599X175-8N, F.Cu at (165.4, 20.3)
- C22, C23: value 2200pF -> 0.1u
- C6: value 1uF -> 0.1u
- J5: value Conn_01x05_Male -> Conn_01x06_Male; footprint Connector_PinHeader_2.54mm:PinHeader_1x05_P2.54mm_Vertical -> Connector_PinSocket_2.54mm:PinSocket_1x06_P2.54mm_Vertical
- R16, R17: value R_LPF -> 10k
- R3: value 500k -> 47k; footprint Resistor_SMD:R_1206_3216Metric -> Resistor_SMD:R_0805_2012Metric
- moved J7 77.1 mm to (118.9, 42.3)
- moved J6 77.1 mm to (116.5, 54.0)
- moved U7 75.2 mm to (122.6, 31.4)
- moved C13 61.3 mm to (163.6, 28.0)
- moved C22 54.1 mm to (168.0, 31.0)
- moved R15 54.1 mm to (168.0, 34.0)
- moved C11 52.2 mm to (167.3, 25.0)
- moved J4 51.3 mm to (134.0, 19.4)
- moved R1 48.7 mm to (166.2, 40.0)
- moved C4 46.9 mm to (162.9, 25.0)
- moved C1 45.7 mm to (163.6, 34.0)
- moved C6 42.5 mm to (154.6, 34.4)
- moved C3 42.3 mm to (159.1, 36.4)
- moved C17 40.3 mm to (168.0, 28.0)
- moved R7 40.3 mm to (161.8, 43.0)
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Connections:
- C22 pad 1: /L_OUT -> /SW3
- C23 pad 1: /R_OUT -> /SW1
- C6 pad 1: Net-(C6-Pad1) -> /CPU_EN
- C6 pad 2: Net-(C6-Pad2) -> GND
- J3 pad 2: /R_OUT -> /C3R_2
- J3 pad 3: /L_OUT -> /C3L_2
- J5 pad 2: /SCK -> Net-(J5-Pad2)
- J5 pad 3: /LRCK -> /SCK_U_I2S
- J5 pad 4: /BCK -> /BCK_U_I2S
- J5 pad 5: /DATA -> /LRCK_U_I2S
- R16 pad 1: /R_OUT -> /SW3
- R16 pad 2: /C3R_2 -> GND
- R17 pad 1: /L_OUT -> /SW1
- R17 pad 2: /C3L_2 -> GND
- R3 pad 1: /+5V -> /+3V3
- R3 pad 2: Net-(R3-Pad2) -> /CPU_EN

Commit message: [Minor] Before order second version (develop)
Parts:
- C11, C12, C13, C14, C15, C16, C21, C8, C9, J1, J5, R10, R11, R12, R13, R14, R15, R4, R5, R6, R7, R8, R9, U3, U5: moved to B.Cu
- moved U4 105.2 mm to (145.8, 124.5), turned to 180 degrees
- moved J5 99.0 mm to (130.6, 118.4), turned to 90 degrees
- moved C6 94.7 mm to (130.6, 126.0), turned to 180 degrees
- moved C5 91.5 mm to (118.4, 112.3)
- moved C19 84.5 mm to (125.0, 112.3), turned to 180 degrees
- moved C18 83.7 mm to (131.1, 112.3)
- moved U3 80.9 mm to (129.5, 99.6), turned to 90 degrees
- moved C17 79.6 mm to (144.8, 104.1)
- moved C8 78.2 mm to (125.0, 109.7)
- moved C11 78.1 mm to (118.9, 86.4), turned to 180 degrees
- moved U6 77.1 mm to (138.0, 106.2)
- moved U7 74.8 mm to (122.4, 106.2), turned to 90 degrees
- moved U1 73.9 mm to (144.3, 100.1)
- moved C1 72.7 mm to (138.2, 102.1)
- moved C4 72.3 mm to (136.7, 92.4), turned to 180 degrees
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Connections:
- net /C1L_1 renamed Net-(C11-Pad1)
- net /C1L_2 renamed Net-(C11-Pad2)
- net /C1R_1 renamed Net-(C14-Pad1)
- net /C1R_2 renamed Net-(C14-Pad2)
- net /C2L_1 renamed Net-(C12-Pad1)
- net /C2R_1 renamed Net-(C15-Pad1)
- net /C3L_1 renamed Net-(C13-Pad2)
- net /C3L_2 renamed /L-CHAN
- net /C3R_1 renamed Net-(C16-Pad2)
- net /C3R_2 renamed /R-CHAN
- net /R1L_1 renamed /VL+
- net /R1R_1 renamed /VR+
- net /R2L_1 renamed /VL-
- net /R2R_1 renamed /VR-
- J2 pad 6: GND -> (no net)
- J2 pad 7: GND -> (no net)
Routing:
- net GND: track 0.00 -> 465.7 mm, vias 0 -> 5
- net /+3V3: track 0.00 -> 239.6 mm, vias 0 -> 2
- net /+VCC: track 0.00 -> 125.0 mm, vias 0 -> 2
- net /+VBAT: track 0.00 -> 102.9 mm, vias 0 -> 1
- net /-VCC: track 0.00 -> 97.3 mm
- net /SW3: track 0.00 -> 96.8 mm, vias 0 -> 3
- net /SW1: track 0.00 -> 91.4 mm, vias 0 -> 3
- net Net-(C1-Pad1): track 0.00 -> 88.5 mm
- net /SW4: track 0.00 -> 86.5 mm, vias 0 -> 3
- net /SW2: track 0.00 -> 70.4 mm, vias 0 -> 3
- net /CPU_+3V3: track 0.00 -> 64.6 mm, vias 0 -> 1
- net /BCK_C_I2S: track 0.00 -> 63.3 mm, vias 0 -> 1
- net /SCK: track 0.00 -> 57.3 mm
- net /LRCK_C_I2S: track 0.00 -> 55.2 mm, vias 0 -> 2
- net /SD_SCK: track 0.00 -> 54.5 mm
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- added copper zone on B.Cu, net GND
- added copper zone on F.Cu, net GND
Other:
- board size 68.1 x 55.9 mm -> 62.5 x 77.7 mm

Commit message: [Minor] 久しぶりの謎コミットなのでバグあるかもしれないです (develop)
Parts:
- removed C22, C23, C24, C25, C6: 0.1u, Capacitor_SMD:C_0805_2012Metric
- removed J7: MEM2067-02-180-00-A_REVB, MEM2067-02-180-00-A_REVB:GCT_MEM2067-02-180-00-A_REVB
- removed R16, R17, R18, R19: 10k, Resistor_SMD:R_0805_2012Metric
- removed R3: 47k, Resistor_SMD:R_0805_2012Metric
- removed S3, S4, S5, S6: 2-1437565-8, 2-1437565-8:SW_2-1437565-8
- removed U4: ESP32-WROOM-32, ESP32-WROOM-32:MODULE_ESP32-WROOM-32
- J4, S1: moved to B.Cu
- J6: value B6B-ZR(LF)(SN) -> Conn_01x06_Male; footprint B6B-ZR_LF_SN:JST_B6B-ZR(LF)(SN) -> Connector_PinSocket_2.54mm:PinSocket_1x06_P2.54mm_Vertical; moved to B.Cu
- moved J5 52.8 mm to (129.5, 65.5), turned to 270 degrees
- moved J6 46.2 mm to (113.3, 79.2)
- moved S2 41.9 mm to (145.8, 90.4), turned to 90 degrees
- moved C19 32.5 mm to (125.4, 79.8), turned to 0 degrees
- moved C17 31.6 mm to (121.4, 82.8), turned to 90 degrees
- moved C5 31.6 mm to (135.6, 85.9), turned to 180 degrees
- moved C20 29.5 mm to (137.2, 108.2), turned to 90 degrees
- moved R2 27.9 mm to (143.8, 71.6), turned to 90 degrees
- moved C18 27.0 mm to (125.5, 85.9)
- moved U6 26.5 mm to (125.6, 82.8)
- moved J4 24.7 mm to (113.3, 97.5), turned to 180 degrees
- moved F1 22.8 mm to (131.1, 71.6), turned to 0 degrees
- moved U2 21.6 mm to (139.7, 71.6), turned to 180 degrees
- moved D1 21.6 mm to (131.1, 75.2), turned to 180 degrees
- moved U7 20.9 mm to (135.6, 89.9), turned to 270 degrees
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Connections:
- J3 pad 2: /R-CHAN -> /L-CHAN
- J3 pad 3: /L-CHAN -> /R-CHAN
- J5 pad 4: /BCK_U_I2S -> /LRCK_U_I2S
- J5 pad 5: /LRCK_U_I2S -> /BCK_U_I2S
- J6 pad 2: /+3V3 -> /CPU_+3V3
- J6 pad 3: /TXD0 -> /SCK_C_I2S
- J6 pad 4: /RXD0 -> /LRCK_C_I2S
- J6 pad 5: /CPU_EN -> /BCK_C_I2S
- J6 pad 6: /BOOT -> /DATA_C_I2S
Routing:
- net GND: track 465.7 -> 246.3 mm, vias 5 -> 12
- net /+3V3: track 239.6 -> 112.5 mm, vias 2 -> 0
- net /SW3: track 96.8 -> 0.00 mm, vias 3 -> 0
- net /SW1: track 91.4 -> 0.00 mm, vias 3 -> 0
- net /SW4: track 86.5 -> 0.00 mm, vias 3 -> 0
- net /SW2: track 70.4 -> 0.00 mm, vias 3 -> 0
- net /SD_SCK: track 54.5 -> 0.00 mm
- net /-VCC: track 97.3 -> 42.9 mm, vias 0 -> 1
- net /CPU_EN: track 54.4 -> 0.00 mm
- net /SCK: track 57.3 -> 19.4 mm
- net Net-(F1-Pad2): track 47.5 -> 12.2 mm
- net /SD_MOSI: track 31.9 -> 0.00 mm
- net Net-(J7-Pad10): track 30.8 -> 0.00 mm
- net /SD_CS: track 29.2 -> 0.00 mm
- net /BOOT: track 27.5 -> 0.00 mm, vias 1 -> 0
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Other:
- board size 62.5 x 77.7 mm -> 40.1 x 70.1 mm
