File: my_first_audio_player.sch (KiCad schematic (older format))
At the start: 57 parts, among them J1 B2B-PH-SM4-TB(LF)(SN), J2 USB3090-XX-X_REVE, J3 SJ-3523-SMT-TR, J4 Conn_01x05_Male, J5 Conn_01x05_Male, J6 Conn 2_10_L, J7 Conn 2_10_R, Q1 SI2333CDS-T1-GE3, U1 ADP150TUJZ3.3-EPR2, U2 MCP73826_4.1VCHCT_ND, U3 PCM1793ADB, U4 LTC3245HMSEPBF, U5 OPA2134, U6 LTC1983ES6-5TRMPBF

Commit message: [Minor] Still not edit Switch, ESP32I2S, PinsocketNumber (develop)
Parts:
- removed C22, C23: 2200pF, Capacitor_SMD:C_0805_2012Metric, symbol Device:C
- removed J6: Conn 2_10_L, SAMTEC-HTSW-110-18-X-D:SAMTEC-HTSW-110-18-X-D, symbol my_first_audio_player-rescue:SAMTEC-HTSW-110-18-X-D-SAMTEC-HTSW-110-18-X-D
- removed J7: Conn 2_10_R, SAMTEC-HTSW-110-18-X-D:SAMTEC-HTSW-110-18-X-D, symbol my_first_audio_player-rescue:SAMTEC-HTSW-110-18-X-D-SAMTEC-HTSW-110-18-X-D
- removed R16, R17: R_LPF, Resistor_SMD:R_0805_2012Metric, symbol Device:R
- removed U4: LTC3245HMSEPBF, LTC3245HMSE:MSOP-12_MSE, symbol my_first_audio_player-rescue:LTC3245HMSEPBF-LTC3245HMSE
- added J6: B6B-ZR(LF)(SN), B6B-ZR_LF_SN:JST_B6B-ZR(LF)(SN), symbol B6B-ZR_LF_SN:B6B-ZR(LF)(SN)
- added J7: MEM2067-02-180-00-A_REVB, GCT_MEM2067-02-180-00-A_REVB, symbol MEM2067-02-180-00-A_REVB:MEM2067-02-180-00-A_REVB
- added S?: SS312SAH4-R, SS312SAH4-R:SW_SS312SAH4-R, symbol my_first_audio_player-rescue:SS312SAH4-R-SS312SAH4-R
- added U4: ESP32-WROOM-32, ESP32-WROOM-32:MODULE_ESP32-WROOM-32, symbol ESP32-WROOM-32:ESP32-WROOM-32
- added U7: ADP150TUJZ3.3-EPR2, ADP151:Analog_Devices-ADP151TUJZ3.3-EPR2-Level_A, symbol my_first_audio_player-rescue:ADP151TUJZ3.3-EPR2-eec
- C6: value 1uF -> 0.1u; footprint Capacitor_SMD:C_0805_2012Metric -> (none)
- C7: value 10uF -> 1uF
- R3: value 500k -> 47k; footprint Resistor_SMD:R_1206_3216Metric -> (none)
Connections:
- net L_OUT is gone; now on net C3L_2: J3.3
- net R_OUT is gone; now on net C3R_2: J3.2
- net +3V3: now also R3.1, J6.2, J7.4 (VDD), S?.2
- net GND: now also C6.2, J6.1, J7.3 (CMD), J7.6 (VSS), U4.1 (GND), U4.15 (GND), U4.38 (GND), U4.39_1 (GND), U4.39_10 (GND), U4.39_11 (GND), U4.39_12 (GND), U4.39_13 (GND), U4.39_14 (GND), U4.39_15 (GND), U4.39_16 (GND), U4.39_17 (GND), U4.39_18 (GND), U4.39_19 (GND), U4.39_2 (GND), U4.39_20 (GND), U4.39_21 (GND), U4.39_3 (GND), U4.39_4 (GND), U4.39_5 (GND), U4.39_6 (GND), U4.39_7 (GND), U4.39_8 (GND), U4.39_9 (GND), U7.2 (GND)
- net at C1.1, C17.1, C5.1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: now also U7.1 (VIN), U7.3 (EN)
- net CPU_EN: now reaches C6.1
- net CPU_EN: now also R3.2, J6.5, U4.3 (EN)
- net +5V renamed +VCC
- net +VCC: now also U7.5 (VOUT); no longer R3.1
- net -5V renamed -VCC
- new net: J7.10 (SHIELD), J7.11 (SHIELD), J7.12 (SHIELD), J7.9 (SHIELD)
- new net BOOT: J6.6, U4.25 (IO0)
- new net CPU_+3V3: S?.1, U4.2 (3V3)
- new net I2S_BCLK: U4.11 (IO26)
- new net I2S_DOUT: U4.31 (IO19)
- new net I2S_LRC: U4.10 (IO25)
- new net RXD0: J6.4, U4.34 (RXD0)
- new net SD_CS: J7.1 (DAT2), U4.16 (IO13)
- new net SD_MISO: J7.7 (DAT0), U4.24 (IO2)
- new net SD_MOSI: J7.2 (CD/DAT3), U4.23 (IO15)
- new net SD_SCK: J7.5 (CLK), U4.13 (IO14)
- new net TXD0: J6.3, U4.35 (TXD0)
- no-connect marks 6 -> 10
Other:
- note added: "2\n"
- note added: "CPU\n"
- note added: "CPU_SWITCH\n\n"
- note added: "Debug Port\n"
- note added: "K001-DAC-V2\n"
- note added: "SD Slot\n"
- note added: "Switch\n"
- note added: "VBAT to +VCC\n"
- note added: "VBAT to -VCC\n"
- note removed: "K001-DAC-V1"
- note removed: "VBAT to +5V"
- note removed: "VBAT to -5V"
- moved on the sheet: C1, C10, C11, C12, C13, C14, C15, C16, C17, C18, C19, C2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

Commit message: [Minor] Maybe create ver2 sch (develop)
Parts:
- removed J5: Conn_01x05_Male, Connector_PinHeader_2.54mm:PinHeader_1x05_P2.54mm_Vertical, symbol Connector:Conn_01x05_Male
- removed S?: SS312SAH4-R, SS312SAH4-R:SW_SS312SAH4-R, symbol my_first_audio_player-rescue:SS312SAH4-R-SS312SAH4-R
- added C22, C23, C24, C25: 0.1u, Capacitor_SMD:C_0805_2012Metric, symbol Device:C
- added J5: Conn_01x06_Male, Connector_PinSocket_2.54mm:PinSocket_1x06_P2.54mm_Vertical, symbol Connector:Conn_01x06_Male
- added R16, R17, R18, R19: 10k, Resistor_SMD:R_0805_2012Metric, symbol Device:R
- added S2: EG6201, EG6201:SW_EG6201, symbol EG6201:EG6201
- added S3, S4, S5, S6: 2-1437565-8, 2-1437565-8:SW_2-1437565-8, symbol 2-1437565-8:2-1437565-8
- C6: footprint (none) -> Capacitor_SMD:C_0805_2012Metric
- J7: footprint GCT_MEM2067-02-180-00-A_REVB -> MEM2067-02-180-00-A_REVB:GCT_MEM2067-02-180-00-A_REVB
- R3: footprint (none) -> Resistor_SMD:R_0805_2012Metric
Connections:
- net +3V3: now also S2.17, S3.1, S3.2, S4.1, S4.2, S5.1, S5.2, S6.1, S6.2
- net BCK: now also S2.8
- net CPU_+3V3: now also S2.18
- net DATA: now also S2.2
- net GND: now also C22.2, C23.2, C24.2, C25.2, J5.1 (Pin_1), R16.2, R17.2, R18.2, R19.2
- net LRCK: now also S2.5
- net SCK: now also S2.11
- net SW1: now reaches U4.27 (IO16)
- net SW1: now also C23.1, R17.1, S4.3, S4.4
- net SW2: now reaches U4.28 (IO17)
- net SW2: now also C25.1, R19.1, S6.3, S6.4
- net SW3: now reaches U4.30 (IO18)
- net SW3: now also C22.1, R16.1, S3.3, S3.4
- net SW4: now reaches U4.33 (IO21)
- net SW4: now also C24.1, R18.1, S5.3, S5.4
- net I2S_BCLK renamed BCK_C_I2S
- net BCK_C_I2S: now also S2.12, S2.9
- net I2S_DOUT renamed DATA_C_I2S
- net DATA_C_I2S: now also S2.3
- net I2S_LRC renamed LRCK_C_I2S
- net LRCK_C_I2S: now also S2.6
- new net: S2.S1 (SHIELD), S2.S2 (SHIELD), S2.S3 (SHIELD), S2.S4 (SHIELD)
- new net BCK_U_I2S: J5.4 (Pin_4), S2.7
- new net DATA_U_I2S: J5.6 (Pin_6), S2.1
- new net LRCK_U_I2S: J5.5 (Pin_5), S2.4
- new net SCK_U_I2S: J5.3 (Pin_3), S2.10
- no-connect marks 10 -> 15
Other:
- note added: "I2S Selector\n"
- note removed: "1"
- note removed: "2\n"
- note removed: "CPU_SWITCH\n\n"
- moved on the sheet: C6, J4, J6, J7, R3, U4

Commit message: [Minor] Before order second version (develop)
Connections:
- net C1L_1: no longer names the net of C11.1, R4.1, R7.2, R8.2
- net C1L_2: no longer names the net of C11.2, R5.1, R6.1, R9.2
- net C1R_1: no longer names the net of C14.1, R10.1, R13.2, R14.2
- net C1R_2: no longer names the net of C14.2, R11.1, R12.1, R15.2
- net C2L_1: no longer names the net of C12.1, R9.1, U5.5 (+)
- net C2R_1: no longer names the net of C15.1, R15.1, U5.3 (+)
- net C3L_1: no longer names the net of C13.2, R8.1, U5.6 (-)
- net C3L_2 renamed L-CHAN
- net C3R_1: no longer names the net of C16.2, R14.1, U5.2 (-)
- net C3R_2 renamed R-CHAN
- net R1L_1 renamed VL+
- net R1R_1 renamed VR+
- net R2L_1 renamed VL-
- net R2R_1 renamed VR-

Commit message: [Minor] 久しぶりの謎コミットなのでバグあるかもしれないです (develop)
Parts:
- removed C22, C23, C24, C25, C6: 0.1u, Capacitor_SMD:C_0805_2012Metric, symbol Device:C
- removed J6: B6B-ZR(LF)(SN), B6B-ZR_LF_SN:JST_B6B-ZR(LF)(SN), symbol B6B-ZR_LF_SN:B6B-ZR(LF)(SN)
- removed J7: MEM2067-02-180-00-A_REVB, MEM2067-02-180-00-A_REVB:GCT_MEM2067-02-180-00-A_REVB, symbol MEM2067-02-180-00-A_REVB:MEM2067-02-180-00-A_REVB
- removed R16, R17, R18, R19: 10k, Resistor_SMD:R_0805_2012Metric, symbol Device:R
- removed R3: 47k, Resistor_SMD:R_0805_2012Metric, symbol Device:R
- removed S3, S4, S5, S6: 2-1437565-8, 2-1437565-8:SW_2-1437565-8, symbol 2-1437565-8:2-1437565-8
- removed U4: ESP32-WROOM-32, ESP32-WROOM-32:MODULE_ESP32-WROOM-32, symbol ESP32-WROOM-32:ESP32-WROOM-32
- added J6: Conn_01x06_Male, Connector_PinSocket_2.54mm:PinSocket_1x06_P2.54mm_Vertical, symbol Connector:Conn_01x06_Male
Connections:
- net BCK_C_I2S: now also J6.5 (Pin_5)
- net BCK_U_I2S: now also J5.5 (Pin_5); no longer J5.4 (Pin_4)
- net CPU_+3V3: now also J6.2 (Pin_2)
- net DATA_C_I2S: now also J6.6 (Pin_6)
- net GND: now also J6.1 (Pin_1)
- net L-CHAN: now also J3.2; no longer J3.3
- net LRCK_C_I2S: now also J6.4 (Pin_4)
- net LRCK_U_I2S: now also J5.4 (Pin_4); no longer J5.5 (Pin_5)
- net R-CHAN: now also J3.3; no longer J3.2
- new net SCK_C_I2S: J6.3 (Pin_3)
- no-connect marks 15 -> 13
Other:
- note removed: "CPU\n"
- note removed: "Debug Port\n"
- note removed: "SD Slot\n"
- note removed: "Switch\n"
- moved on the sheet: J4, J5, S2
